Commit message: change message type into PointCloud2

File: urdf/livox_mid40.xacro (robot description, xacro)
@@ -6,5 +6,5 @@
   <xacro:property name="horizontal_fov" value="38.4"/>
   <xacro:property name="vertical_fov" value="38.4"/>
-  <xacro:property name="ros_topic" value="scan"/>
+  <xacro:property name="ros_topic" value="livox_lidar/livox"/>
   <xacro:property name="samples" value="10000"/>
   <xacro:property name="downsample" value="1"/>

Commit message: add use_inf method.

File: urdf/livox_mid40.xacro (robot description, xacro)
@@ -3,5 +3,5 @@
   <xacro:property name="M_PI" value="3.14159"/>
   <xacro:property name="laser_min_range" value="0.1"/>
-  <xacro:property name="laser_max_range" value="200.0"/>
+  <xacro:property name="laser_max_range" value="100.0"/>
   <xacro:property name="horizontal_fov" value="38.4"/>
   <xacro:property name="vertical_fov" value="38.4"/>
@@ -9,4 +9,5 @@
   <xacro:property name="samples" value="10000"/>
   <xacro:property name="downsample" value="1"/>
+  <xacro:property name="use_inf" value="false"/>
   <xacro:macro name="null_inertial">
     <inertial>
@@ -55,4 +56,5 @@
 		  <downsample>${downsample}</downsample>
 		  <csv_file_name>package://livox_laser_simulation/scan_mode/mid40.csv</csv_file_name>
+      <use_inf>${use_inf}</use_inf>
 		  <ros_topic>${ros_topic}</ros_topic>
         </plugin>
