Commit message: update livox_ros_dirver::CustomMsg.

File: urdf/livox_gazebo_sensor.xacro (robot description, xacro)
@@ -4,7 +4,7 @@
     <inertial>
       <mass value="0.1"/>
-    <inertia ixx="0.01" ixy="0" ixz="0"
-          iyy="0.01" iyz="0"
-          izz="0.01"/>
+    <inertia ixx="0.001" ixy="0" ixz="0"
+          iyy="0.001" iyz="0"
+          izz="0.001"/>
     </inertial>
   </xacro:macro>
@@ -13,5 +13,5 @@
       <sensor type="ray" name="laser_${name}">
         <pose>0 0 0 0 0 0</pose>
-        <visualize>${visualize}</visualize>
+        <visualize>True</visualize>
         <update_rate>${update_rate}</update_rate>
         <!-- This ray plgin is only for visualization. -->

File: urdf/livox_horizon.xacro (robot description, xacro)
@@ -6,15 +6,14 @@
   <xacro:property name="horizontal_fov" value="81.7"/>
   <xacro:property name="vertical_fov" value="25.1"/>
-  <xacro:property name="ros_topic" value="scan"/>
+  <xacro:property name="ros_topic" value="livox/lidar"/>
   <xacro:property name="samples" value="24000"/>
-  <xacro:property name="downsample" value="1"/>
   <xacro:property name="publish_pointcloud_type" value="0"/>
   <xacro:property name="csv_file_name" value="package://livox_laser_simulation/scan_mode/horizon.csv"/>
   <xacro:include filename="$(find livox_laser_simulation)/urdf/livox_gazebo_sensor.xacro"/>
-  <xacro:macro name="Livox_Horizon" params="visualize:=True name:=livox publish_pointcloud_type:=0 ros_topic:=scan">
+  <xacro:macro name="Livox_Horizon" params="visualize:=True name:=livox publish_pointcloud_type:=0 ros_topic:=livox/lidar downsample:=1">
     <link name="${name}_base">
       <xacro:null_inertial/>
       <visual>
-        <origin xyz="0.00 0 0.00" rpy="0 0 0"/>
+        <origin xyz="0.07 0 0.05" rpy="0 0 0"/>
         <geometry>
           <mesh filename="package://livox_laser_simulation/meshes/livox_mid40.dae">
@@ -23,7 +22,9 @@
       </visual>
       <collision>
-		  <origin xyz="0 0 0" rpy="0 0 0" /> <geometry> <mesh
-		  filename="package://livox_laser_simulation/meshes/livox_mid40.dae">
-		  </mesh> </geometry>
+		  <origin xyz="0.07 0 0.05" rpy="0 0 0" />
+      <geometry>
+        <mesh filename="package://livox_laser_simulation/meshes/livox_mid40.dae">
+		    </mesh>
+      </geometry>
       </collision>
     </link>

File: urdf/robot.xacro (robot description, xacro)
@@ -2,5 +2,5 @@
 <robot xmlns:xacro="http://ros.org/wiki/xacro">
   <xacro:include filename="$(find livox_laser_simulation)/urdf/livox_horizon.xacro"/>
-  <Livox_Horizon name="livox" visualize="true" publish_pointcloud_type="2"/>
+  <Livox_Horizon name="livox" visualize="true" publish_pointcloud_type="3" downsample="1"/>
   <xacro:include filename="$(find livox_laser_simulation)/urdf/standardrobots_oasis300.xacro"/>
   <xacro:link_oasis name="oasis"/>

Commit message: change point tag

File: urdf/livox_gazebo_sensor.xacro (robot description, xacro)
@@ -52,16 +52,16 @@
       <sensor name="livox_imu" type="imu">
         <always_on>true</always_on>
-        <update_rate>50</update_rate>
+        <update_rate>200</update_rate>
         <visualize>false</visualize>
         <topic>"/livox/imu"</topic>
         <plugin filename="libgazebo_ros_imu_sensor.so" name="imu_plugin">
           <topicName>/livox/imu</topicName>
-          <bodyName>imu_link</bodyName>
-          <updateRateHZ>10.0</updateRateHZ>
+          <bodyName>livox_imu_link</bodyName>
+          <updateRateHZ>200.0</updateRateHZ>
           <xyzOffset>0 0 0</xyzOffset>
           <!-- <gaussianNoise>0.0026399240948208127</gaussianNoise> -->
           <gaussianNoise>0.00</gaussianNoise>
           <rpyOffset>0 0 0</rpyOffset>
-          <frameName>imu_link</frameName>
+          <frameName>livox_imu_link</frameName>
           <initialOrientationAsReference>false</initialOrientationAsReference>
         </plugin>

File: urdf/livox_horizon.xacro (robot description, xacro)
@@ -15,5 +15,5 @@
       <xacro:null_inertial/>
       <visual>
-        <origin xyz="0.07 0 0.05" rpy="0 0 0"/>
+        <origin xyz="0.00 0 0.00" rpy="0 0 0"/>
         <geometry>
           <mesh filename="package://livox_laser_simulation/meshes/livox_mid40.dae">
@@ -22,5 +22,5 @@
       </visual>
       <collision>
-		  <origin xyz="0.07 0 0.05" rpy="0 0 0" />
+		  <origin xyz="0.00 0 0.00" rpy="0 0 0" />
       <geometry>
         <mesh filename="package://livox_laser_simulation/meshes/livox_mid40.dae">
@@ -37,4 +37,10 @@
       <origin rpy="0 0 0" xyz="0.0 0.0 0.0"/>
     </joint>
+    <link name="${name}_imu_link"/>
+    <joint name="imu_link_joint" type="fixed">
+      <parent link="${name}"/>
+      <child link="${name}_imu_link"/>
+      <origin rpy="0 0 0" xyz="-0.05512 -0.02226 0.0297"/>
+    </joint>
     <xacro:Livox_gazebo_sensor name="${name}" visualize="${visualize}" publish_pointcloud_type="${publish_pointcloud_type}"/>
   </xacro:macro>

Commit message: Fix noise in IMU plugin
Signed-off-by: Emiliano Borghi <emiliano@smartmachine.nz>

File: urdf/livox_gazebo_sensor.xacro (robot description, xacro)
@@ -9,5 +9,8 @@
     </inertial>
   </xacro:macro>
-  <xacro:macro name="Livox_gazebo_sensor" params="visualize:=True update_rate:=10 resolution:=0.002 noise_mean:=0.0 noise_stddev:=0.01 name:=livox publish_pointcloud_type:=1">
+  <xacro:macro name="Livox_gazebo_sensor"
+               params="visualize:=True update_rate:=10 resolution:=0.002
+                       noise_mean:=0.0 noise_stddev:=0.01 imu_noise_stddev:=0.0026399240948208127
+                       name:=livox publish_pointcloud_type:=1">
     <gazebo reference="${name}">
       <sensor type="ray" name="livox_lidar">
@@ -21,12 +24,12 @@
             <samples>100</samples>
             <resolution>1</resolution>
-            <min_angle>${-horizontal_fov/360*M_PI}</min_angle>
-            <max_angle>${horizontal_fov/360*M_PI}</max_angle>
+            <min_angle>${-horizontal_fov/360*pi}</min_angle>
+            <max_angle>${horizontal_fov/360*pi}</max_angle>
             </horizontal>
             <vertical>
             <samples>50</samples>
             <resolution>1</resolution>
-            <min_angle>${-vertical_fov/360*M_PI}</min_angle>
-            <max_angle>${vertical_fov/360*M_PI}</max_angle>
+            <min_angle>${-vertical_fov/360*pi}</min_angle>
+            <max_angle>${vertical_fov/360*pi}</max_angle>
             </vertical>
             </scan>
@@ -51,8 +54,8 @@
       </sensor>
       <sensor name="livox_imu" type="imu">
+        <pose>0 0 0 0 0 0</pose>
         <always_on>true</always_on>
         <update_rate>200</update_rate>
         <visualize>false</visualize>
-        <topic>"/livox/imu"</topic>
         <plugin filename="libgazebo_ros_imu_sensor.so" name="imu_plugin">
           <topicName>/livox/imu</topicName>
@@ -60,11 +63,9 @@
           <updateRateHZ>200.0</updateRateHZ>
           <xyzOffset>0 0 0</xyzOffset>
-          <!-- <gaussianNoise>0.0026399240948208127</gaussianNoise> -->
-          <gaussianNoise>0.00</gaussianNoise>
+          <gaussianNoise>${imu_noise_stddev}</gaussianNoise>
           <rpyOffset>0 0 0</rpyOffset>
           <frameName>livox_imu_link</frameName>
           <initialOrientationAsReference>false</initialOrientationAsReference>
         </plugin>
-        <pose>0 0 0 0 0 0</pose>
       </sensor>
     </gazebo>
