Commit message: add line information into point.

File: urdf/livox_horizon.xacro (robot description, xacro)
@@ -9,56 +9,8 @@
   <xacro:property name="samples" value="24000"/>
   <xacro:property name="downsample" value="1"/>
-  <xacro:macro name="null_inertial">
-    <inertial>
-      <mass value="0.1"/>
-    <inertia ixx="0.01" ixy="0" ixz="0"
-          iyy="0.01" iyz="0"
-          izz="0.01"/>
-    </inertial>
-  </xacro:macro>
-  <xacro:macro name="Livox_Mid_gazebo_sensor" params="visualize:=True update_rate:=10 resolution:=0.002 noise_mean:=0.0 noise_stddev:=0.01 name:=livox">
-    <gazebo reference="${name}">
-      <sensor type="ray" name="laser_${name}">
-        <pose>0 0 0 0 0 0</pose>
-        <visualize>${visualize}</visualize>
-        <update_rate>${update_rate}</update_rate>
-        <!-- This ray plgin is only for visualization. -->
-        <plugin name="gazebo_ros_laser_controller" filename="liblivox_laser_simulation.so">
-			<ray>
-			  <scan>
-				<horizontal>
-				<samples>100</samples>
-				<resolution>1</resolution>
-				<min_angle>${-horizontal_fov/360*M_PI}</min_angle>
-				<max_angle>${horizontal_fov/360*M_PI}</max_angle>
-				</horizontal>
-				<vertical>
-				<samples>50</samples>
-				<resolution>1</resolution>
-				<min_angle>${-vertical_fov/360*M_PI}</min_angle>
-				<max_angle>${vertical_fov/360*M_PI}</max_angle>
-				</vertical>
-			  </scan>
-			  <range>
-				<min>${laser_min_range}</min>
-				<max>${laser_max_range}</max>
-				<resolution>${resolution}</resolution>
-			  </range>
-			  <noise>
-				<type>gaussian</type>
-				<mean>${noise_mean}</mean>
-				<stddev>${noise_stddev}</stddev>
-			  </noise>
-			</ray>
-          <visualize>${visualize}</visualize>
-		  <samples>${samples}</samples>
-		  <downsample>${downsample}</downsample>
-		  <csv_file_name>package://livox_laser_simulation/scan_mode/horizon.csv</csv_file_name>
-		  <ros_topic>${ros_topic}</ros_topic>
-        </plugin>
-      </sensor>
-    </gazebo>
-  </xacro:macro>
-  <xacro:macro name="Livox_HORIZON" params="visualize:=True name:=livox">
+  <xacro:property name="publish_pointcloud_type" value="0"/>
+  <xacro:property name="csv_file_name" value="package://livox_laser_simulation/scan_mode/horizon.csv"/>
+  <xacro:include filename="$(find livox_laser_simulation)/urdf/livox_gazebo_sensor.xacro"/>
+  <xacro:macro name="Livox_Horizon" params="visualize:=True name:=livox publish_pointcloud_type:=0">
     <link name="${name}_base">
       <xacro:null_inertial/>
@@ -84,8 +36,5 @@
       <origin rpy="0 0 0" xyz="0.0 0.0 0.0"/>
     </joint>
-    <xacro:Livox_Mid_gazebo_sensor name="${name}" visualize="${visualize}"/>
+    <xacro:Livox_gazebo_sensor name="${name}" visualize="${visualize}" publish_pointcloud_type="${publish_pointcloud_type}"/>
   </xacro:macro>
-    <xacro:Livox_HORIZON name="livox"/>
-  <xacro:include filename="$(find livox_laser_simulation)/urdf/standardrobots_oasis300.xacro"/>
-  <xacro:link_oasis name="oasis"/>
 </robot>

File: urdf/livox_mid40.xacro (robot description, xacro)
@@ -9,56 +9,8 @@
   <xacro:property name="samples" value="10000"/>
   <xacro:property name="downsample" value="1"/>
-  <xacro:macro name="null_inertial">
-    <inertial>
-      <mass value="0.1"/>
-    <inertia ixx="0.01" ixy="0" ixz="0"
-          iyy="0.01" iyz="0"
-          izz="0.01"/>
-    </inertial>
-  </xacro:macro>
-  <xacro:macro name="Livox_Mid_gazebo_sensor" params="visualize:=True update_rate:=10 resolution:=0.002 noise_mean:=0.0 noise_stddev:=0.01 name:=livox">
-    <gazebo reference="${name}">
-      <sensor type="ray" name="laser_${name}">
-        <pose>0 0 0 0 0 0</pose>
-        <visualize>${visualize}</visualize>
-        <update_rate>${update_rate}</update_rate>
-        <!-- This ray plgin is only for visualization. -->
-        <plugin name="gazebo_ros_laser_controller" filename="liblivox_laser_simulation.so">
-			<ray>
-			  <scan>
-				<horizontal>
-				<samples>100</samples>
-				<resolution>1</resolution>
-				<min_angle>${-horizontal_fov/360*M_PI}</min_angle>
-				<max_angle>${horizontal_fov/360*M_PI}</max_angle>
-				</horizontal>
-				<vertical>
-				<samples>50</samples>
-				<resolution>1</resolution>
-				<min_angle>${-vertical_fov/360*M_PI}</min_angle>
-				<max_angle>${vertical_fov/360*M_PI}</max_angle>
-				</vertical>
-			  </scan>
-			  <range>
-				<min>${laser_min_range}</min>
-				<max>${laser_max_range}</max>
-				<resolution>${resolution}</resolution>
-			  </range>
-			  <noise>
-				<type>gaussian</type>
-				<mean>${noise_mean}</mean>
-				<stddev>${noise_stddev}</stddev>
-			  </noise>
-			</ray>
-          <visualize>${visualize}</visualize>
-		  <samples>${samples}</samples>
-		  <downsample>${downsample}</downsample>
-		  <csv_file_name>package://livox_laser_simulation/scan_mode/mid40.csv</csv_file_name>
-		  <ros_topic>${ros_topic}</ros_topic>
-        </plugin>
-      </sensor>
-    </gazebo>
-  </xacro:macro>
-  <xacro:macro name="Livox_Mid40" params="visualize:=True name:=livox">
+  <xacro:property name="publish_pointcloud_type" value="0"/>
+  <xacro:property name="csv_file_name" value="package://livox_laser_simulation/scan_mode/mid40.csv"/>
+  <xacro:include filename="$(find livox_laser_simulation)/urdf/livox_gazebo_sensor.xacro"/>
+  <xacro:macro name="Livox_Mid40" params="visualize:=True name:=livox publish_pointcloud_type:=1">
     <link name="${name}_base">
       <xacro:null_inertial/>
@@ -86,8 +38,5 @@
       <origin rpy="0 0 0" xyz="0.0 0.0 0.0"/>
     </joint>
-    <xacro:Livox_Mid_gazebo_sensor name="${name}" visualize="${visualize}"/>
+    <xacro:Livox_gazebo_sensor name="${name}" visualize="${visualize}"/>
   </xacro:macro>
-  <!-- <xacro:Livox_Mid40 name="livox"/>
-  <xacro:include filename="$(find livox_laser_simulation)/urdf/standardrobots_oasis300.xacro"/>
-  <xacro:link_oasis name="oasis"/> -->
 </robot>

Commit message: fix bugs of timestamp and point range.

File: urdf/livox_horizon.xacro (robot description, xacro)
@@ -12,5 +12,5 @@
   <xacro:property name="csv_file_name" value="package://livox_laser_simulation/scan_mode/horizon.csv"/>
   <xacro:include filename="$(find livox_laser_simulation)/urdf/livox_gazebo_sensor.xacro"/>
-  <xacro:macro name="Livox_Horizon" params="visualize:=True name:=livox publish_pointcloud_type:=0">
+  <xacro:macro name="Livox_Horizon" params="visualize:=True name:=livox publish_pointcloud_type:=0 ros_topic:=scan">
     <link name="${name}_base">
       <xacro:null_inertial/>

File: urdf/livox_mid40.xacro (robot description, xacro)
@@ -12,5 +12,5 @@
   <xacro:property name="csv_file_name" value="package://livox_laser_simulation/scan_mode/mid40.csv"/>
   <xacro:include filename="$(find livox_laser_simulation)/urdf/livox_gazebo_sensor.xacro"/>
-  <xacro:macro name="Livox_Mid40" params="visualize:=True name:=livox publish_pointcloud_type:=1">
+  <xacro:macro name="Livox_Mid40" params="visualize:=True name:=livox publish_pointcloud_type:=1 ros_topic:=scan">
     <link name="${name}_base">
       <xacro:null_inertial/>

Commit message: update sensor_msg.

File: urdf/livox_horizon.xacro (robot description, xacro)
@@ -6,63 +6,14 @@
   <xacro:property name="horizontal_fov" value="81.7"/>
   <xacro:property name="vertical_fov" value="25.1"/>
-  <xacro:property name="ros_topic" value="scan"/>
+  <xacro:property name="ros_topic" value="livox/lidar"/>
   <xacro:property name="samples" value="24000"/>
-  <xacro:property name="downsample" value="1"/>
-  <xacro:macro name="null_inertial">
-    <inertial>
-      <mass value="0.1"/>
-    <inertia ixx="0.01" ixy="0" ixz="0"
-          iyy="0.01" iyz="0"
-          izz="0.01"/>
-    </inertial>
-  </xacro:macro>
-  <xacro:macro name="Livox_Mid_gazebo_sensor" params="visualize:=True update_rate:=10 resolution:=0.002 noise_mean:=0.0 noise_stddev:=0.01 name:=livox">
-    <gazebo reference="${name}">
-      <sensor type="ray" name="laser_${name}">
-        <pose>0 0 0 0 0 0</pose>
-        <visualize>${visualize}</visualize>
-        <update_rate>${update_rate}</update_rate>
-        <!-- This ray plgin is only for visualization. -->
-        <plugin name="gazebo_ros_laser_controller" filename="liblivox_laser_simulation.so">
-			<ray>
-			  <scan>
-				<horizontal>
-				<samples>100</samples>
-				<resolution>1</resolution>
-				<min_angle>${-horizontal_fov/360*M_PI}</min_angle>
-				<max_angle>${horizontal_fov/360*M_PI}</max_angle>
-				</horizontal>
-				<vertical>
-				<samples>50</samples>
-				<resolution>1</resolution>
-				<min_angle>${-vertical_fov/360*M_PI}</min_angle>
-				<max_angle>${vertical_fov/360*M_PI}</max_angle>
-				</vertical>
-			  </scan>
-			  <range>
-				<min>${laser_min_range}</min>
-				<max>${laser_max_range}</max>
-				<resolution>${resolution}</resolution>
-			  </range>
-			  <noise>
-				<type>gaussian</type>
-				<mean>${noise_mean}</mean>
-				<stddev>${noise_stddev}</stddev>
-			  </noise>
-			</ray>
-          <visualize>${visualize}</visualize>
-		  <samples>${samples}</samples>
-		  <downsample>${downsample}</downsample>
-		  <csv_file_name>package://livox_laser_simulation/scan_mode/horizon.csv</csv_file_name>
-		  <ros_topic>${ros_topic}</ros_topic>
-        </plugin>
-      </sensor>
-    </gazebo>
-  </xacro:macro>
-  <xacro:macro name="Livox_HORIZON" params="visualize:=True name:=livox">
+  <xacro:property name="publish_pointcloud_type" value="0"/>
+  <xacro:property name="csv_file_name" value="package://livox_laser_simulation/scan_mode/horizon.csv"/>
+  <xacro:include filename="$(find livox_laser_simulation)/urdf/livox_gazebo_sensor.xacro"/>
+  <xacro:macro name="Livox_Horizon" params="visualize:=True name:=livox publish_pointcloud_type:=0 ros_topic:=livox/lidar downsample:=1">
     <link name="${name}_base">
       <xacro:null_inertial/>
       <visual>
-        <origin xyz="0.00 0 0.00" rpy="0 0 0"/>
+        <origin xyz="0.07 0 0.05" rpy="0 0 0"/>
         <geometry>
           <mesh filename="package://livox_laser_simulation/meshes/livox_mid40.dae">
@@ -71,7 +22,9 @@
       </visual>
       <collision>
-		  <origin xyz="0 0 0" rpy="0 0 0" /> <geometry> <mesh
-		  filename="package://livox_laser_simulation/meshes/livox_mid40.dae">
-		  </mesh> </geometry>
+		  <origin xyz="0.07 0 0.05" rpy="0 0 0" />
+      <geometry>
+        <mesh filename="package://livox_laser_simulation/meshes/livox_mid40.dae">
+		    </mesh>
+      </geometry>
       </collision>
     </link>
@@ -84,8 +37,5 @@
       <origin rpy="0 0 0" xyz="0.0 0.0 0.0"/>
     </joint>
-    <xacro:Livox_Mid_gazebo_sensor name="${name}" visualize="${visualize}"/>
+    <xacro:Livox_gazebo_sensor name="${name}" visualize="${visualize}" publish_pointcloud_type="${publish_pointcloud_type}"/>
   </xacro:macro>
-    <xacro:Livox_HORIZON name="livox"/>
-  <xacro:include filename="$(find livox_laser_simulation)/urdf/standardrobots_oasis300.xacro"/>
-  <xacro:link_oasis name="oasis"/>
 </robot>

File: urdf/livox_mid40.xacro (robot description, xacro)
@@ -3,64 +3,14 @@
   <xacro:property name="M_PI" value="3.14159"/>
   <xacro:property name="laser_min_range" value="0.1"/>
-  <xacro:property name="laser_max_range" value="100.0"/>
+  <xacro:property name="laser_max_range" value="200.0"/>
   <xacro:property name="horizontal_fov" value="38.4"/>
   <xacro:property name="vertical_fov" value="38.4"/>
-  <xacro:property name="ros_topic" value="livox_lidar/livox"/>
+  <xacro:property name="ros_topic" value="scan"/>
   <xacro:property name="samples" value="10000"/>
   <xacro:property name="downsample" value="1"/>
-  <xacro:property name="use_inf" value="false"/>
-  <xacro:macro name="null_inertial">
-    <inertial>
-      <mass value="0.1"/>
-    <inertia ixx="0.01" ixy="0" ixz="0"
-          iyy="0.01" iyz="0"
-          izz="0.01"/>
-    </inertial>
-  </xacro:macro>
-  <xacro:macro name="Livox_Mid_gazebo_sensor" params="visualize:=True update_rate:=10 resolution:=0.002 noise_mean:=0.0 noise_stddev:=0.01 name:=livox">
-    <gazebo reference="${name}">
-      <sensor type="ray" name="laser_${name}">
-        <pose>0 0 0 0 0 0</pose>
-        <visualize>${visualize}</visualize>
-        <update_rate>${update_rate}</update_rate>
-        <!-- This ray plgin is only for visualization. -->
-        <plugin name="gazebo_ros_laser_controller" filename="liblivox_laser_simulation.so">
-			<ray>
-			  <scan>
-				<horizontal>
-				<samples>100</samples>
-				<resolution>1</resolution>
-				<min_angle>${-horizontal_fov/360*M_PI}</min_angle>
-				<max_angle>${horizontal_fov/360*M_PI}</max_angle>
-				</horizontal>
-				<vertical>
-				<samples>50</samples>
-				<resolution>1</resolution>
-				<min_angle>${-vertical_fov/360*M_PI}</min_angle>
-				<max_angle>${vertical_fov/360*M_PI}</max_angle>
-				</vertical>
-			  </scan>
-			  <range>
-				<min>${laser_min_range}</min>
-				<max>${laser_max_range}</max>
-				<resolution>${resolution}</resolution>
-			  </range>
-			  <noise>
-				<type>gaussian</type>
-				<mean>${noise_mean}</mean>
-				<stddev>${noise_stddev}</stddev>
-			  </noise>
-			</ray>
-          <visualize>${visualize}</visualize>
-		  <samples>${samples}</samples>
-		  <downsample>${downsample}</downsample>
-		  <csv_file_name>package://livox_laser_simulation/scan_mode/mid40.csv</csv_file_name>
-      <use_inf>${use_inf}</use_inf>
-		  <ros_topic>${ros_topic}</ros_topic>
-        </plugin>
-      </sensor>
-    </gazebo>
-  </xacro:macro>
-  <xacro:macro name="Livox_Mid40" params="visualize:=True name:=livox">
+  <xacro:property name="publish_pointcloud_type" value="0"/>
+  <xacro:property name="csv_file_name" value="package://livox_laser_simulation/scan_mode/mid40.csv"/>
+  <xacro:include filename="$(find livox_laser_simulation)/urdf/livox_gazebo_sensor.xacro"/>
+  <xacro:macro name="Livox_Mid40" params="visualize:=True name:=livox publish_pointcloud_type:=1 ros_topic:=scan">
     <link name="${name}_base">
       <xacro:null_inertial/>
@@ -88,8 +38,5 @@
       <origin rpy="0 0 0" xyz="0.0 0.0 0.0"/>
     </joint>
-    <xacro:Livox_Mid_gazebo_sensor name="${name}" visualize="${visualize}"/>
+    <xacro:Livox_gazebo_sensor name="${name}" visualize="${visualize}"/>
   </xacro:macro>
-  <!-- <xacro:Livox_Mid40 name="livox"/>
-  <xacro:include filename="$(find livox_laser_simulation)/urdf/standardrobots_oasis300.xacro"/>
-  <xacro:link_oasis name="oasis"/> -->
 </robot>

Commit message: Modify Livox Horizon noise via Xacro arguments
Signed-off-by: Emiliano Borghi <emiliano@smartmachine.nz>

File: urdf/livox_horizon.xacro (robot description, xacro)
@@ -11,5 +11,6 @@
   <xacro:property name="csv_file_name" value="package://livox_laser_simulation/scan_mode/horizon.csv"/>
   <xacro:include filename="$(find livox_laser_simulation)/urdf/livox_gazebo_sensor.xacro"/>
-  <xacro:macro name="Livox_Horizon" params="visualize:=True name:=livox publish_pointcloud_type:=0 ros_topic:=livox/lidar downsample:=1">
+  <xacro:macro name="Livox_Horizon" params="visualize:=True name:=livox publish_pointcloud_type:=0 ros_topic:=livox/lidar downsample:=1
+                                            noise_mean:=0.0 noise_stddev:=0.01 imu_noise_stddev:=0.0026399240948208127">
     <link name="${name}_base">
       <xacro:null_inertial/>
@@ -43,5 +44,6 @@
       <origin rpy="0 0 0" xyz="-0.05512 -0.02226 0.0297"/>
     </joint>
-    <xacro:Livox_gazebo_sensor name="${name}" visualize="${visualize}" publish_pointcloud_type="${publish_pointcloud_type}"/>
+    <xacro:Livox_gazebo_sensor name="${name}" visualize="${visualize}" publish_pointcloud_type="${publish_pointcloud_type}"
+                               noise_mean="${noise_mean}" noise_stddev="${noise_stddev}" imu_noise_stddev="${imu_noise_stddev}"/>
   </xacro:macro>
 </robot>
